File: Pure SH.sch (EAGLE design)
At the start: 26 parts, among them T1 3904, U1 LF398, U2 4093

Commit message: SandH 1.1
Parts:
- added R7: 0R, rcl:R-US_R0805
- R2: value 10K -> 2K2***
Connections:
- net +12V: now also R7.2
- net N$3: now also R7.1
Other:
- moved on the sheet: U$1G$1
Changed lines of the file:
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@@
 <part name="T1" library="QuBit" deviceset="TRANSISTOR_MMBT3904" device="" value="3904"/>
 <part name="R1" library="rcl" deviceset="R-US_" device="R0805" value="100K"/>
-<part name="R2" library="rcl" deviceset="R-US_" device="R0805" value="10K"/>
+<part name="R2" library="rcl" deviceset="R-US_" device="R0805" value="2K2***"/>
 <part name="R3" library="rcl" deviceset="R-US_" device="R0805" value="10K"/>
 <part name="R4" library="rcl" deviceset="R-US_" device="R0805" value="1K"/>
@@
 <part name="C7" library="rcl" deviceset="C-US" device="C0805K" value="1u"/>
 <part name="U$1" library="INSTRUO" deviceset="LED_RG_SMD_REV" device=""/>
+<part name="R7" library="rcl" deviceset="R-US_" device="R0805" value="0R"/>
 </parts>
 <sheets>
@@
 <instance part="GND1" gate="1" x="35.56" y="40.64"/>
 <instance part="GND2" gate="1" x="60.96" y="40.64"/>
-<instance part="SUPPLY1" gate="+12V" x="60.96" y="114.3"/>
+<instance part="SUPPLY1" gate="+12V" x="60.96" y="116.84"/>
 <instance part="GND3" gate="1" x="121.92" y="55.88"/>
 <instance part="SUPPLY2" gate="+12V" x="220.98" y="96.52"/>
@@
 <instance part="R6" gate="G$1" x="-7.62" y="20.32" rot="R180"/>
 <instance part="C7" gate="G$1" x="-40.64" y="-5.08"/>
-<instance part="U$1" gate="G$1" x="60.96" y="104.14"/>
+<instance part="U$1" gate="G$1" x="60.96" y="106.68"/>
 <instance part="U$1" gate="G$2" x="83.82" y="104.14"/>
+<instance part="R7" gate="G$1" x="48.26" y="104.14" rot="R90"/>
 </instances>
 <busses>
@@
 <segment>
 <pinref part="SUPPLY1" gate="+12V" pin="+12V"/>
-<wire x1="60.96" y1="106.68" x2="60.96" y2="111.76" width="0.1524" layer="91"/>
+<wire x1="60.96" y1="109.22" x2="60.96" y2="111.76" width="0.1524" layer="91"/>
 <pinref part="U$1" gate="G$1" pin="A"/>
+<wire x1="60.96" y1="111.76" x2="60.96" y2="114.3" width="0.1524" layer="91"/>
+<junction x="60.96" y="111.76"/>
+<pinref part="R7" gate="G$1" pin="2"/>
+<wire x1="60.96" y1="111.76" x2="48.26" y2="111.76" width="0.1524" layer="91"/>
+<wire x1="48.26" y1="111.76" x2="48.26" y2="109.22" width="0.1524" layer="91"/>
 </segment>
 <segment>
@@
 <segment>
 <pinref part="R2" gate="G$1" pin="2"/>
-<wire x1="60.96" y1="99.06" x2="60.96" y2="93.98" width="0.1524" layer="91"/>
+<wire x1="60.96" y1="101.6" x2="60.96" y2="96.52" width="0.1524" layer="91"/>
 <pinref part="U$1" gate="G$1" pin="C"/>
-</segment>
-</net>
+<wire x1="60.96" y1="96.52" x2="60.96" y2="93.98" width="0.1524" layer="91"/>
+<junction x="60.96" y="96.52"/>
+<pinref part="R7" gate="G$1" pin="1"/>
+<wire x1="60.96" y1="96.52" x2="48.26" y2="96.52" width="0.1524" layer="91"/>
+<wire x1="48.26" y1="96.52" x2="48.26" y2="99.06" width="0.1524" layer="91"/>
+</segment>
+</net>

Commit message: SandH 1.2
Parts:
- removed R7: 0R, rcl:R-US_R0805
- removed U$1: LED_RG_SMD_REV, INSTRUO:LED_RG_SMD_REV
- added C10, C8: 0.1u, rcl:C-USC0805K
- added IC1: TL072D, linear:TL072D
- added R10: 100K, rcl:R-US_R0805
- added R8, R9: 100k, rcl:R-US_R0805
Connections:
- removed net N$3: R2.2, R7.1, U$1G$1.C
- new net N$12: IC1A.-IN, R5.1, R8.2
- new net N$16: IC1A.OUT, R8.1, U1.IN
- new net N$17: R10.2, U1.OUT
- new net N$18: IC1B.-IN, R10.1, R9.2
- new net N$19: IC1B.OUT, OUT.TIP, R9.1
- new net N$21: C8.1, IC1P.V+
- net +12V: now also R2.2; no longer R7.2, U$1G$1.A
- net GND: now also C10.1, C8.2, IC1A.+IN, IC1B.+IN; no longer R5.1
- net N$11: no longer U1.IN
- net N$20: now also C10.2, IC1P.V-; no longer OUT.TIP, U1.OUT
Other:
- note removed: "10K"
- moved on the sheet: IN, OUT, R5

Commit message: SandH 1.3
Parts:
- removed U2: 4093, QuBit:4093
- added IC2: 4093D, 40xx:4093D
Connections:
- removed net N$20: C10.2, IC1P.V-
- removed net N$21: C8.1, IC1P.V+
- net +12V: now also C8.1, IC1P.V+, IC2P.VDD; no longer U2G$1.+12V
- net -12V: now also C10.2, IC1P.V-
- net GND: now also IC2P.VSS
- net N$14: now also IC2B.I0, IC2B.I1; no longer U2G$4.I1, U2G$4.I2
- net N$15: now also IC2B.O; no longer U2G$4.O
- net N$4: now also IC2D.I0, IC2D.I1; no longer U2G$6.I1, U2G$6.I2
- net N$5: now also IC2D.O; no longer U2G$6.O
- net N$7: now also IC2C.I0, IC2C.I1; no longer U2G$5.I1, U2G$5.I2
- net N$8: now also IC2A.I0, IC2A.I1, IC2C.O; no longer U2G$3.I1, U2G$3.I2, U2G$5.O
- net N$9: now also IC2A.O; no longer U2G$3.O

Commit message: SandH 1.4
Parts:
- removed U1: LF398, QuBit:LF398
- added C11: 100nF, GMSN:CAPACITOR-USC0805
- added IC3: cd4093, GMSN:SCHMITT_TRIG_QUAD
- added R7: 1k, GMSN:RESISTOR_USR0805
- C1, C7: device rcl:C-USC0805K -> GMSN:CAPACITOR-USC0805
- C10, C3, C6, C8, C9: value 0.1u -> 100nF; device rcl:C-USC0805K -> GMSN:CAPACITOR-USC0805
- C2: value 0.1u -> Polypropylene Film 4.7nF; device rcl:C-USC0805K -> GMSN:CAPACITOR-US050-045X075
- C4, C5: value 10u -> 10uF; device rcl:CPOL-US153CLV-0505 -> GMSN:CAPACITOR_POL-US153CLV-0505
- CLK, IN, OUT: value S_JACK -> PJ301M-12; device INSTRUO:S_JACK -> GMSN:SOCKET_MONO_3.5MMPJ301M-12
- D1: device SparkFun-DiscreteSemi:DIODESOD -> GMSN:DIODEDO-41
- D2, D3: value (none) -> STTH102A; device adafruit:DIODESMA -> GMSN:DIODEDO-41
- IC1: value TL072D -> LF398; device linear:TL072D -> GMSN:SAMPLE_HOLD_LF398
- IC2: value 4093D -> TL072; device 40xx:4093D -> GMSN:OPAMP_DUALD
- PWR: value M05X2SHD -> HEADER2X5SHD; device SparkFun-Connectors:M05X2SHD -> GMSN:HEADER2X5SHD
- R1, R10, R5: value 100K -> 100k; device rcl:R-US_R0805 -> GMSN:RESISTOR_USR0805
- R2: value 2K2*** -> 2K2; device rcl:R-US_R0805 -> GMSN:RESISTOR_USR0805
- R3: value 10K -> 10k; device rcl:R-US_R0805 -> GMSN:RESISTOR_USR0805
- R4: value 1K -> 5k6; device rcl:R-US_R0805 -> GMSN:RESISTOR_USR0805
- R6: value 2K2 -> 2k2; device rcl:R-US_R0805 -> GMSN:RESISTOR_USR0805
- R8, R9: device rcl:R-US_R0805 -> GMSN:RESISTOR_USR0805
- RATE: device QuBit:Q-POT -> GMSN:RESISTOR_VARIABLE9MM_POT
- T1: value 3904 -> MMBT3904; device QuBit:TRANSISTOR_MMBT3904 -> GMSN:TRANSISTOR_NPNSOT23
Connections:
- removed net N$8: IC2A.I0, IC2A.I1, IC2C.O
- new net N$3: C1.1, IC3G$6.O
- net +12V: now also C11.1, IC1.V+, IC2P.V+, IC3G$1.V+; no longer IC1P.V+, IC2P.VDD, U1.V+
- net -12V: now also IC1.V-, IC2P.V-; no longer IC1P.V-, U1.V-
- net GND: now also C11.2, CLK.SLEEVE, IC1.GND, IC2A.+IN, IC2B.+IN, IC3G$1.V-, IN.SLEEVE, OUT.SLEEVE, R7.1; no longer CLK.GND, IC1A.+IN, IC1B.+IN, IC2P.VSS, IN.GND, OUT.GND, U1.GND
- net N$10: now also IC1.CAP; no longer U1.CAP
- net N$12: now also IC2A.-IN; no longer IC1A.-IN
- net N$14: now also IC3G$4.I1, IC3G$4.I2; no longer IC2B.I0, IC2B.I1
- net N$15: now also CLK.SWITCH, IC3G$4.O; no longer CLK.NORM, IC2B.O
- net N$16: now also IC1.IN, IC2A.OUT; no longer IC1A.OUT, U1.IN
- net N$17: now also IC1.OUT; no longer U1.OUT
- net N$18: now also IC2B.-IN; no longer IC1B.-IN
- net N$19: now also IC2B.OUT; no longer IC1B.OUT
- net N$4: now also IC3G$6.I1, IC3G$6.I2; no longer IC2D.I0, IC2D.I1
- net N$5: now also IC3G$3.I1, IC3G$3.I2, IC3G$5.O; no longer C1.1, IC2D.O
- net N$6: now also IC1.CLKIN, R7.2; no longer U1.CLKIN
- net N$7: now also IC3G$5.I1, IC3G$5.I2; no longer IC2C.I0, IC2C.I1
- net N$9: now also IC3G$3.O; no longer IC2A.O
Other:
- note removed: "100K"
- moved on the sheet: R3, R4

Commit message: SandH 1.5
S&H Updated to V1.5 14/4/21

Library updated to include 3D models.
Traces rerouted.
Parts:
- C2: device GMSN:CAPACITOR-US050-045X075 -> GMSN:CAPACITOR-USC050-045X075
- D2, D3: device GMSN:DIODEDO-41 -> GMSN:DIODESMA

Commit message: Reinstall
Parts:
- R10, R5, R8, R9: value 100k -> 10k
- R2: value 2K2 -> 2k2
- RATE: value Q-POT -> A1M
